File: designs/u-blox-MAX-F10S-00B/hardware/u-blox-MAX-F10S-00B.kicad_sch (KiCad schematic)
At the start: 21 parts, among them IC101 MAX-F10S-00B, J102 PRT-14417, J103 PRT-14417, J104 Conn_01x07_Pin, J105 Conn_Coaxial_Small, J106 Conn_Coaxial_Small, J107 Conn_02x05_Counter_Clockwise, U101 MIC5318YMT-TR

Commit message: pcb done?
Parts:
- J6: renamed from J104; footprint Connector_PinHeader_2.54mm:PinHeader_1x07_P2.54mm_Vertical -> Connector_PinHeader_2.54mm:PinHeader_1x07_P2.54mm_Vertical_SMD_Pin1Left
- U1: renamed from IC101; footprint pcb-u-blox:MAXF10S00B -> MAXF10S00B
- renumbered C102 to C1, C101 to C2, C103 to C3, C104 to C4, C105 to C5, H101 to H1, H102 to H2, H103 to H3, H104 to H4, J105 to J1, J106 to J2, J107 to J3, J102 to J4, J103 to J5, R103 to R1, R104 to R2, R102 to R3, R101 to R4, U101 to U2
Other:
- moved on the sheet: J3, J4, J5, J6, R3, R4

Commit message: switched to m3 holes
Parts:
- H1, H2, H3, H4: footprint MountingHole:MountingHole_2.2mm_M2_Pad_Via -> MountingHole:MountingHole_3.2mm_M3_Pad_Via
Changed lines of the file:
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@@
 			)
 		)
-		(property "Footprint" "MountingHole:MountingHole_2.2mm_M2_Pad_Via"
+		(property "Footprint" "MountingHole:MountingHole_3.2mm_M3_Pad_Via"
 			(at 77.47 167.64 0)
 			(hide yes)
@@
 			)
 		)
-		(property "Footprint" "MountingHole:MountingHole_2.2mm_M2_Pad_Via"
+		(property "Footprint" "MountingHole:MountingHole_3.2mm_M3_Pad_Via"
 			(at 68.58 167.64 0)
 			(hide yes)
@@
 			)
 		)
-		(property "Footprint" "MountingHole:MountingHole_2.2mm_M2_Pad_Via"
+		(property "Footprint" "MountingHole:MountingHole_3.2mm_M3_Pad_Via"
 			(at 95.25 167.64 0)
 			(hide yes)
@@
 			)
 		)
-		(property "Footprint" "MountingHole:MountingHole_2.2mm_M2_Pad_Via"
+		(property "Footprint" "MountingHole:MountingHole_3.2mm_M3_Pad_Via"
 			(at 86.36 167.64 0)
 			(hide yes)
