File: designs/u-blox-MAX-F10S-00B/hardware/_restore_backup_2026-05-14T21-09-39-204/u-blox-MAX-F10S-00B.kicad_sch (KiCad schematic)
At the start: 21 parts, among them IC101 MAX-F10S-00B, J102 PRT-14417, J103 PRT-14417, J104 Conn_01x07_Pin, J105 Conn_Coaxial_Small, J106 Conn_Coaxial_Small, J107 Conn_02x05_Counter_Clockwise, U101 MIC5318YMT-TR

Commit message: need to check pad to pad clearance of jlcpcb
Parts:
- U101: footprint TMLF-6_MT_MCH -> pcb-MicrochipTechnology:MIC5318YMT-TR
Connections:
- net EXTINT: now also J104.4 (Pin_4); no longer J104.6 (Pin_6)
- net GND: no longer U101.7 (EPAD)
- net RESET_N: now also J104.6 (Pin_6); no longer J104.4 (Pin_4)
- net SAFEBOOT_N: now also J104.7 (Pin_7); no longer J104.3 (Pin_3)
- net TIMEPULSE: now also J104.3 (Pin_3); no longer J104.7 (Pin_7)
Changed lines of the file:
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@@
 	(wire
 		(pts
-			(xy 63.5 45.72) (xy 63.5 46.99)
-		)
-		(stroke
-			(width 0)
-			(type default)
-		)
-	)
-	(wire
-		(pts
 			(xy 81.28 171.45) (xy 86.36 171.45)
 		)
@@
 	)
 	(label "RESET_N"
-		(at 250.19 129.54 180)
+		(at 250.19 124.46 180)
 		(effects
 			(font
@@
 	)
 	(label "TIMEPULSE"
-		(at 250.19 121.92 180)
+		(at 250.19 132.08 180)
 		(effects
 			(font
@@
 	)
 	(label "SAFEBOOT_N"
-		(at 250.19 132.08 180)
+		(at 250.19 121.92 180)
 		(effects
 			(font
@@
 	)
 	(label "EXTINT"
-		(at 250.19 124.46 180)
+		(at 250.19 129.54 180)
 		(effects
 			(font
@@
 			)
 		)
-		(property "Footprint" "TMLF-6_MT_MCH"
+		(property "Footprint" "pcb-MicrochipTechnology:MIC5318YMT-TR"
 			(at 42.164 21.336 0)
 			(hide yes)
@@
 		(pin "6"
 		)
-		(pin "7"
-		)
 		(instances
 			(project "u-blox-MAX-F10S-00B"
@@
 					(unit 1)
 				)
-			)
-		)
-	)
-	(symbol
-		(lib_id "power:GND")
-		(at 63.5 46.99 0)
-		(unit 1)
-		(body_style 1)
-		(exclude_from_sim no)
-		(in_bom yes)
-		(on_board yes)
-		(in_pos_files yes)
-		(dnp no)
-		(fields_autoplaced yes)
-		(property "Reference" "#PWR0122"
-			(at 63.5 53.34 0)
-			(hide yes)
-			(show_name no)
-			(do_not_autoplace no)
-			(effects
-				(font
-					(size 1.27 1.27)
-				)
-			)
-		)
-		(property "Value" "GND"
-			(at 63.5 52.07 0)
-			(show_name no)
-			(do_not_autoplace no)
-			(effects
-				(font
-					(size 1.27 1.27)
-				)
-			)
-		)
-		(property "Footprint" ""
-			(at 63.5 46.99 0)
-			(hide yes)
-			(show_name no)
-			(do_not_autoplace no)
-			(effects
-				(font
-					(size 1.27 1.27)
-				)
-			)
-		)
-		(property "Datasheet" ""
-			(at 63.5 46.99 0)
-			(hide yes)
-			(show_name no)
-			(do_not_autoplace no)
-			(effects
-				(font
-					(size 1.27 1.27)
-				)
-			)
-		)
-		(property "Description" "Power symbol creates a global label with name \"GND\" , ground"
-			(at 63.5 46.99 0)
-			(hide yes)
-			(show_name no)
-			(do_not_autoplace no)
-			(effects
-				(font
-					(size 1.27 1.27)
-				)
-			)
-		)
-		(pin "1"
-		)
-		(instances
-			(project "u-blox-MAX-F10S-00B"
-				(path "/42e1d221-83dd-4a9a-aabf-76b26236b056"
-					(reference "#PWR0122")
-					(unit 1)
-				)
