File: designs/ftdi-FT232RNQ/hardware/ftdi-FT232RNQ.kicad_sch (KiCad schematic)
At the start: 0 parts

Commit message: schematic done
Parts:
- added C1, C3, C5: 100n, Capacitor_SMD:C_0402_1005Metric, symbol Device:C
- added C2, C4: 4u7, Capacitor_SMD:C_0402_1005Metric, symbol Device:C
- added D1, D2: LED, Diode_SMD:D_0402_1005Metric, symbol Device:LED
- added H1, H2, H3, H4: MountingHole_Pad, MountingHole:MountingHole_3.2mm_M3_Pad_Via, symbol Mechanical:MountingHole_Pad
- added J1: Conn_02x05_Odd_Even, Connector_IDC:IDC-Header_2x05_P2.54mm_Vertical_SMD, symbol Connector_Generic:Conn_02x05_Odd_Even
- added J2: USB_C_Receptacle_USB2.0_14P, Connector_USB:USB_C_Receptacle_GCT_USB4110, symbol Connector:USB_C_Receptacle_USB2.0_14P
- added J3, J4: Conn_01x03_Pin, Connector_PinHeader_2.54mm:PinHeader_1x03_P2.54mm_Vertical_SMD_Pin1Left, symbol Connector:Conn_01x03_Pin
- added R1, R2: 4k7, Resistor_SMD:R_0402_1005Metric, symbol Device:R
- added R3, R4: 270, Resistor_SMD:R_0402_1005Metric, symbol Device:R
- added R5, R6: 5k1, Resistor_SMD:R_0402_1005Metric, symbol Device:R
- added U1: FT232RNQ, pcb-FTDI:FT232RNQ, symbol pcb-FTDI:FT232RNQ
- added U2: ESDR0502NMUTBG, pcb-onsemi:ESDR0502NMUTBG, symbol pcb-onsemi:ESDR0502NMUTBG
Connections:
- new net: J2.A6 (D+), J2.B6 (D+), U1.14 (USBDP), U2.5 (D+)
- new net: J2.A7 (D-), J2.B7 (D-), U1.15 (USBDM), U2.4 (D-)
- new net: D2.2 (A), R4.2
- new net: D1.2 (A), R3.2
- new net: J2.A5 (CC1), R6.1
- new net: J2.B5 (CC2), R5.1
- new net +3V3: C1.1, J3.1 (Pin_1), U1.16 (3V3OUT)
- new net +5V: C2.1, C3.1, C4.1, C5.1, J1.10 (Pin_10), J2.A4 (VBUS), J2.A9 (VBUS), J2.B4 (VBUS), J2.B9 (VBUS), J3.3 (Pin_3), R1.1, R3.1, R4.1, U1.19 (VCC), U2.6 (VBUS)
- new net CBUS0/TXLED#: D1.1 (K), U1.22 (CBUS0)
- new net CBUS1/RXLED#: D2.1 (K), U1.21 (CBUS1)
- new net CBUS2/TXDEN: J4.1 (Pin_1), U1.10 (CBUS2)
- new net CBUS3/PWREN#: J4.2 (Pin_2), U1.11 (CBUS3)
- new net CBUS4/SLEEP#: J4.3 (Pin_3), U1.9 (CBUS4)
- new net CTS#: J1.8 (Pin_8), U1.8 (CTS#)
- new net DCD#: J1.1 (Pin_1), U1.7 (DCD#)
- new net DSR#: J1.6 (Pin_6), U1.6 (DSR#)
- new net DTR#: J1.4 (Pin_4), U1.31 (DTR#)
- new net GND: C1.2, C2.2, C3.2, C4.2, C5.2, H1.1, H2.1, H3.1, H4.1, J1.5 (Pin_5), J2.A1 (GND), J2.A12 (GND), J2.B1 (GND), J2.B12 (GND), J2.SH (SHIELD), R2.2, R5.2, R6.2, U1.17 (GND), U1.20 (GND), U1.24 (AGND), U1.33 (EP/GND), U1.4 (GND), U2.1 (GND)
- new net RESET#: R1.2, U1.18 (RESET#)
- new net RI#: J1.9 (Pin_9), U1.3 (RI#)
- new net RTS#: J1.7 (Pin_7), U1.32 (RTS#)
- new net RXD: J1.2 (Pin_2), U1.2 (RXD)
- new net TEST: R2.1, U1.26 (TEST)
- new net TXD: J1.3 (Pin_3), U1.30 (TXD)
- new net VCCIO: J3.2 (Pin_2), U1.1 (VCCIO)
- no-connect marks 0 -> 10
Other:
- note added: "pull to gnd?"
