File: designs/ftdi-FT232RNQ/hardware/ftdi-FT232RNQ.kicad_sch (KiCad schematic)
At the start: 23 parts, among them J1 Conn_02x05_Odd_Even, J2 USB_C_Receptacle_USB2.0_14P, J3 Conn_01x03_Pin, J4 Conn_01x03_Pin, U1 FT232RNQ, U2 ESDR0502NMUTBG

Commit message: latice
Connections:
- net USB_+: now reaches J2.A6 (D+), J2.B6 (D+), U1.14 (USBDP), U2.5 (D+)
- net USB_+: now also U2.2 (NC)
- net USB_-: now reaches J2.A7 (D-), J2.B7 (D-), U1.15 (USBDM), U2.4 (D-)
- net USB_-: now also U2.3 (NC)
- net CC1: now reaches J2.A5 (CC1), R6.1
- net CC2: now reaches J2.B5 (CC2), R5.1
- no-connect marks 10 -> 8
Changed lines of the file:
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@@
 	)
 	(no_connect
-		(at 43.18 110.49)
-	)
-	(no_connect
-		(at 43.18 107.95)
-	)
-	(no_connect
 		(at 123.19 90.17)
 	)
@@
 	(wire
 		(pts
+			(xy 41.91 107.95) (xy 43.18 107.95)
+		)
+		(stroke
+			(width 0)
+			(type default)
+		)
+	)
+	(wire
+		(pts
 			(xy 168.91 80.01) (xy 170.18 80.01)
 		)
@@
 	(wire
 		(pts
+			(xy 41.91 110.49) (xy 43.18 110.49)
+		)
+		(stroke
+			(width 0)
+			(type default)
+		)
+	)
+	(wire
+		(pts
 			(xy 27.94 96.52) (xy 27.94 97.79)
 		)
@@
 	(wire
 		(pts
-			(xy 43.18 105.41) (xy 38.1 105.41)
+			(xy 43.18 105.41) (xy 29.21 105.41)
 		)
 		(stroke
@@
 	(wire
 		(pts
-			(xy 38.1 105.41) (xy 38.1 109.22)
+			(xy 29.21 105.41) (xy 29.21 109.22)
 		)
 		(stroke
@@
 		)
 	)
+	(label "USB_-"
+		(at 105.41 69.85 180)
+		(effects
+			(font
+				(size 1.27 1.27)
+			)
+			(justify right bottom)
+		)
+	)
 	(label "CBUS2{slash}TXDEN"
 		(at 152.4 171.45 90)
@@
 		)
 	)
+	(label "USB_+"
+		(at 41.91 107.95 180)
+		(effects
+			(font
+				(size 1.27 1.27)
+			)
+			(justify right bottom)
+		)
+	)
 	(label "DTR#"
 		(at 250.19 82.55 0)
@@
 		)
 	)
+	(label "CC1"
+		(at 57.15 67.31 0)
+		(effects
+			(font
+				(size 1.27 1.27)
+			)
+			(justify left bottom)
+		)
+	)
 	(label "DTR#"
 		(at 170.18 72.39 0)
@@
 		)
 	)
+	(label "USB_+"
+		(at 105.41 74.93 180)
+		(effects
+			(font
+				(size 1.27 1.27)
+			)
+			(justify right bottom)
+		)
+	)
 	(label "CTS#"
 		(at 170.18 69.85 0)
@@
 		)
 	)
+	(label "USB_-"
+		(at 41.91 110.49 180)
+		(effects
+			(font
+				(size 1.27 1.27)
+			)
+			(justify right bottom)
+		)
+	)
 	(label "CBUS1{slash}RXLED#"
 		(at 170.18 90.17 0)
@@
 		)
 	)
+	(label "CC2"
+		(at 49.53 67.31 0)
+		(effects
+			(font
+				(size 1.27 1.27)
+			)
+			(justify left bottom)
+		)
+	)
 	(symbol
 		(lib_id "power:+5V")
@@
 	(symbol
 		(lib_id "power:GND")
-		(at 38.1 109.22 0)
+		(at 29.21 109.22 0)
 		(unit 1)
 		(body_style 1)
@@
 		(fields_autoplaced yes)
 		(property "Reference" "#PWR015"
-			(at 38.1 115.57 0)
+			(at 29.21 115.57 0)
 			(hide yes)
 			(show_name no)
@@
 		)
 		(property "Value" "GND"
-			(at 38.1 114.3 0)
+			(at 29.21 114.3 0)
 			(show_name no)
 			(do_not_autoplace no)
@@
 		)
 		(property "Footprint" ""
-			(at 38.1 109.22 0)
+			(at 29.21 109.22 0)
 			(hide yes)
 			(show_name no)
@@
 		)
 		(property "Datasheet" ""
-			(at 38.1 109.22 0)
+			(at 29.21 109.22 0)
 			(hide yes)
 			(show_name no)
@@
 		)
 		(property "Description" "Power symbol creates a global label with name \"GND\" , ground"
-			(at 38.1 109.22 0)
+			(at 29.21 109.22 0)
 			(hide yes)
 			(show_name no)
