File: designs/ftdi-FT232RNQ/hardware/ftdi-FT232RNQ.kicad_pcb (KiCad board)
At the start: 4 copper layers, 40 x 40 mm, 19 parts, among them J1 Conn_02x05_Odd_Even, J2 USB_C_Receptacle_USB2.0_14P, U1 FT232RNQ, U2 ESDR0502NMUTBG

Commit message: latice
Parts:
- added J3: Conn_01x03_Pin, Connector_PinHeader_2.54mm:PinHeader_1x03_P2.54mm_Vertical_SMD_Pin1Left, F.Cu at (143.4, 109.3)
- added J4: Conn_01x03_Pin, Connector_PinHeader_2.54mm:PinHeader_1x03_P2.54mm_Vertical_SMD_Pin1Left, F.Cu at (150.0, 116.6)
- added R5: 5k1, Resistor_SMD:R_0402_1005Metric, F.Cu at (138.9, 102.5)
- added R6: 5k1, Resistor_SMD:R_0402_1005Metric, F.Cu at (138.9, 97.7)
- H1, H2, H3, H4: footprint MountingHole:MountingHole_2.2mm_M2_Pad_Via -> MountingHole:MountingHole_3.2mm_M3_Pad_Via
- moved J1 63.4 mm to (163.2, 100.0)
- moved H4 62.5 mm to (165.0, 85.0)
- moved H3 55.2 mm to (165.0, 115.0)
- moved C5 43.5 mm to (157.5, 108.0), turned to 90 degrees
- moved C4 42.4 mm to (156.6, 108.0), turned to 90 degrees
- moved U1 39.8 mm to (150.0, 100.0), turned to -90 degrees
- moved R2 39.5 mm to (154.0, 101.3)
- moved D1 38.1 mm to (151.8, 104.1), turned to -90 degrees
- moved R3 37.4 mm to (151.8, 106.0), turned to 90 degrees
- moved J2 36.8 mm to (133.7, 100.0), turned to -90 degrees
- moved D2 36.8 mm to (150.9, 104.1), turned to -90 degrees
- moved R4 36.4 mm to (150.9, 106.0), turned to 90 degrees
- moved C3 35.7 mm to (149.5, 103.7)
- moved C2 35.3 mm to (149.5, 104.6)
- moved U2 34.7 mm to (144.7, 100.5)
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Connections:
- J2 pad A5: unconnected-(J2-CC1-PadA5) -> /CC1
- J2 pad A6: Net-(U1-USBDP) -> /USB_+
- J2 pad A7: Net-(U1-USBDM) -> /USB_-
- J2 pad B5: unconnected-(J2-CC2-PadB5) -> /CC2
- J2 pad B6: Net-(U1-USBDP) -> /USB_+
- J2 pad B7: Net-(U1-USBDM) -> /USB_-
- U1 pad 1: +3V3 -> /VCCIO
- U1 pad 14: Net-(U1-USBDP) -> /USB_+
- U1 pad 15: Net-(U1-USBDM) -> /USB_-
- U2 pad 2: unconnected-(U2-NC-Pad2) -> /USB_+
- U2 pad 3: unconnected-(U2-NC-Pad3) -> /USB_-
- U2 pad 4: Net-(U1-USBDM) -> /USB_-
- U2 pad 5: Net-(U1-USBDP) -> /USB_+
Other:
- board text added: "+3V3"
- board text added: "+5V"
- board text added: "VCCIO"
