File: designs/lattice-iCE40UP5K-SG48I/_restore_backup_2026-07-09T22-41-17-153/lattice-iCE40UP5K-SG48I.kicad_pcb (KiCad board)
At the start: 4 copper layers, 70 x 40 mm, 88 parts, among them J1 USB_C_Receptacle_USB2.0_14P, J2 PRT-14417, J3 Conn_01x02, J4 Conn_01x07, J5 Conn_02x06_Top_Bottom, J6 Conn_02x06_Top_Bottom, J7 Conn_02x06_Top_Bottom, J8 Conn_02x06_Top_Bottom, U1 RTQ2520GQW, U2 RTQ2520GQW, U3 ICE40UP5K-SG48I, U4 FT2232HQ, U5 ESDR0502NMUTBG, U6 AT93C46DN-SH-B, U7 BY25Q40GWTIG, X1 DSC6003JI2B

Commit message: temp
Parts:
- added R24: 10k, Resistor_SMD:R_0402_1005Metric, F.Cu at (113.3, 89.9)
- moved C36 83.4 mm to (98.9, 89.7), turned to 0 degrees
- moved C19 73.9 mm to (96.0, 81.8), turned to 0 degrees
- moved C20 72.6 mm to (96.0, 83.8), turned to 0 degrees
- moved C34 72.1 mm to (98.9, 81.8), turned to 0 degrees
- moved C35 70.9 mm to (98.9, 83.8), turned to 0 degrees
- moved C23 70.7 mm to (98.9, 77.9), turned to 0 degrees
- moved C17 70.4 mm to (96.0, 79.9), turned to 0 degrees
- moved C18 70.3 mm to (96.0, 77.9), turned to 0 degrees
- moved C24 69.7 mm to (98.9, 79.9), turned to 0 degrees
- moved C29 63.8 mm to (96.0, 91.7), turned to 0 degrees
- moved C28 63.6 mm to (96.0, 89.7), turned to 0 degrees
- moved R15 63.4 mm to (113.3, 99.8), turned to 0 degrees
- moved C22 62.8 mm to (96.0, 87.7), turned to 0 degrees
- moved C21 62.7 mm to (96.0, 85.8), turned to 0 degrees
- moved R16 62.5 mm to (116.2, 87.9), turned to 0 degrees
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- renumbered J4 to J2, J5 to J3, J6 to J4, J7 to J5, J8 to J6, J2 to J7, J3 to J8
Connections:
- U4 pad 59: +3V3 -> /PWRSAV#
Routing:
- removed copper zone on F.Cu, net GND
- removed copper zone on In2.Cu, net GND
Other:
- board text removed: "LABEL PMOD PINS"
