File: designs/lattice-iCE40UP5K-SG48I/_restore_backup_2026-07-09T22-41-17-153/lattice-iCE40UP5K-SG48I.kicad_sch (KiCad schematic)
At the start: 89 parts, among them J1 USB_C_Receptacle_USB2.0_14P, J2 PRT-14417, J3 Conn_01x02, J4 Conn_01x07, J5 Conn_02x06_Top_Bottom, J6 Conn_02x06_Top_Bottom, J7 Conn_02x06_Top_Bottom, J8 Conn_02x06_Top_Bottom, SW1 SW_MEC_5G, U1 RTQ2520GQW, U2 RTQ2520GQW, U3 ICE40UP5K-SG48I, U4 FT2232HQ, U5 ESDR0502NMUTBG, U6 AT93C46DN-SH-B, U7 BY25Q40GWTIG, X1 DSC6003JI2B

Commit message: temp
Parts:
- added R24: 10k, Resistor_SMD:R_0402_1005Metric, symbol Device:R
Connections:
- net +3V3: now also R24.1; no longer U4.59 (BCBUS7)
- new net PWRSAV#: R24.2, U4.59 (BCBUS7)
Changed lines of the file:
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@@
 	(wire
 		(pts
+			(xy 281.94 191.77) (xy 281.94 190.5)
+		)
+		(stroke
+			(width 0)
+			(type default)
+		)
+	)
+	(wire
+		(pts
 			(xy 259.08 161.29) (xy 259.08 162.56)
 		)
@@
 	(wire
 		(pts
-			(xy 261.62 190.5) (xy 261.62 191.77)
-		)
-		(stroke
-			(width 0)
-			(type default)
-		)
-	)
-	(wire
-		(pts
 			(xy 537.21 209.55) (xy 535.94 209.55)
 		)
@@
 	(wire
 		(pts
+			(xy 248.92 191.77) (xy 281.94 191.77)
+		)
+		(stroke
+			(width 0)
+			(type default)
+		)
+	)
+	(wire
+		(pts
 			(xy 232.41 100.33) (xy 232.41 101.6)
 		)
@@
 	(wire
 		(pts
-			(xy 248.92 191.77) (xy 261.62 191.77)
-		)
-		(stroke
-			(width 0)
-			(type default)
-		)
-	)
-	(wire
-		(pts
 			(xy 524.51 100.33) (xy 524.51 99.06)
 		)
@@
 	(wire
 		(pts
+			(xy 281.94 181.61) (xy 281.94 182.88)
+		)
+		(stroke
+			(width 0)
+			(type default)
+		)
+	)
+	(wire
+		(pts
 			(xy 90.17 38.1) (xy 90.17 33.02)
 		)
@@
 	)
 	(symbol
+		(lib_id "Device:R")
+		(at 281.94 186.69 0)
+		(unit 1)
+		(body_style 1)
+		(exclude_from_sim no)
+		(in_bom yes)
+		(on_board yes)
+		(in_pos_files yes)
+		(dnp no)
+		(fields_autoplaced yes)
+		(property "Reference" "R24"
+			(at 284.48 185.4199 0)
+			(show_name no)
+			(do_not_autoplace no)
+			(effects
+				(font
+					(size 1.27 1.27)
+				)
+				(justify left)
+			)
+		)
+		(property "Value" "10k"
+			(at 284.48 187.9599 0)
+			(show_name no)
+			(do_not_autoplace no)
+			(effects
+				(font
+					(size 1.27 1.27)
+				)
+				(justify left)
+			)
+		)
+		(property "Footprint" "Resistor_SMD:R_0402_1005Metric"
+			(at 280.162 186.69 90)
+			(hide yes)
+			(show_name no)
+			(do_not_autoplace no)
+			(effects
+				(font
+					(size 1.27 1.27)
+				)
+			)
+		)
+		(property "Datasheet" ""
+			(at 281.94 186.69 0)
+			(hide yes)
+			(show_name no)
+			(do_not_autoplace no)
+			(effects
+				(font
+					(size 1.27 1.27)
+				)
+			)
+		)
+		(property "Description" "Resistor"
+			(at 281.94 186.69 0)
+			(hide yes)
+			(show_name no)
+			(do_not_autoplace no)
+			(effects
+				(font
+					(size 1.27 1.27)
+				)
+			)
+		)
+		(pin "1"
+		)
+		(pin "2"
+		)
+		(instances
+			(project "lattice-iCE40UP5K-SG48I"
+				(path "/e0a68d80-6b92-4ac2-8789-569b9c117dc1"
+					(reference "R24")
+					(unit 1)
+				)
+			)
+		)
+	)
+	(symbol
 		(lib_id "power:GND")
 		(at 186.69 48.26 0)
@@
 	(symbol
 		(lib_id "power:+1V8")
-		(at 261.62 190.5 0)
+		(at 281.94 181.61 0)
 		(unit 1)
 		(body_style 1)
@@
 		(dnp no)
 		(property "Reference" "#PWR070"
-			(at 261.62 194.31 0)
+			(at 281.94 185.42 0)
 			(hide yes)
 			(show_name no)
@@
 		)
 		(property "Value" "+3V3"
-			(at 261.62 186.69 0)
+			(at 281.94 177.8 0)
 			(show_name no)
 			(do_not_autoplace no)
@@
 		)
 		(property "Footprint" ""
-			(at 261.62 190.5 0)
+			(at 281.94 181.61 0)
 			(hide yes)
 			(show_name no)
@@
 		)
 		(property "Datasheet" ""
-			(at 261.62 190.5 0)
+			(at 281.94 181.61 0)
 			(hide yes)
 			(show_name no)
@@
 		)
 		(property "Description" "Power symbol creates a global label with name \"+1V8\""
-			(at 261.62 190.5 0)
+			(at 281.94 181.61 0)
 			(hide yes)
 			(show_name no)
