File: designs/lattice-iCE40UP5K-SG48I/lattice-iCE40UP5K-SG48I.kicad_pcb (KiCad board)
At the start: 4 copper layers, 70 x 40 mm, 88 parts, among them J1 USB_C_Receptacle_USB2.0_14P, J2 PRT-14417, J3 Conn_01x02, J4 Conn_01x07, J5 Conn_02x06_Top_Bottom, J6 Conn_02x06_Top_Bottom, J7 Conn_02x06_Top_Bottom, J8 Conn_02x06_Top_Bottom, U1 RTQ2520GQW, U2 RTQ2520GQW, U3 ICE40UP5K-SG48I, U4 FT2232HQ, U5 ESDR0502NMUTBG, U6 AT93C46DN-SH-B, U7 BY25Q40GWTIG, X1 DSC6003JI2B

Commit message: save
Parts:
- J5, J6, J7, J8: footprint Connector_PinHeader_2.54mm:PinHeader_2x06_P2.54mm_Vertical_SMD -> pcb-Samtec:SAMTEC-SMH-106-02-X-D
- moved C36 57.9 mm to (126.6, 81.3), turned to 45 degrees
- moved J2 51.5 mm to (182.5, 93.4), turned to 90 degrees
- moved U6 50.7 mm to (129.6, 84.2), turned to 135 degrees
- moved R16 50.6 mm to (128.2, 87.5)
- moved R24 45.9 mm to (178.1, 93.9), turned to 0 degrees
- moved R15 44.5 mm to (132.1, 87.6), turned to -135 degrees
- moved J4 42.4 mm to (129.6, 71.8), turned to -90 degrees
- moved R19 42.2 mm to (133.4, 86.3), turned to -135 degrees
- moved R14 42.2 mm to (133.9, 84.4), turned to 135 degrees
- moved J3 33.9 mm to (129.8, 115.0), turned to -90 degrees
- moved R22 25.5 mm to (152.9, 88.5), turned to -135 degrees
- moved R23 25.0 mm to (148.0, 95.1), turned to 45 degrees
- moved J6 24.3 mm to (149.9, 114.1), turned to 180 degrees
- moved C37 23.2 mm to (149.8, 88.2), turned to -135 degrees
- moved U7 23.2 mm to (147.4, 92.2), turned to 45 degrees
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- renumbered R25 to R24
Other:
- board size 70 x 40 mm -> 70 x 50 mm
- board text added: "+3V3"
- board text added: "GND"
