File: designs/lattice-iCE40UP5K-SG48I/lattice-iCE40UP5K-SG48I.kicad_pcb (KiCad board)
At the start: 6 copper layers, 70 x 50 mm, 101 parts, among them J1 Conn_Coaxial_Small, J2 USB_C_Receptacle_USB2.0_14P, J4 PRT-14417, J5 Conn_02x06_Top_Bottom, J6 Conn_02x06_Top_Bottom, J7 Conn_01x02, J8 Conn_01x07, J9 Conn_02x06_Top_Bottom, U1 RTQ2520GQW, U2 RTQ2520GQW, U3 ICE40UP5K-SG48I, U4 FT2232HQ, U5 ESDR0502NMUTBG, U6 AT93C46DN-SH-B, U7 BY25Q40GWTIG, X1 DSC6003JI2B, X2 DSC6003JI2B

Commit message: ??
Parts:
- removed the U5 at (126.7, 95.0)
- added D3: D_TVS, Diode_SMD:D_SOD-523, F.Cu at (124.2, 97.2)
- added D4: D_TVS, Diode_SMD:D_SOD-523, F.Cu at (126.1, 92.6)
- added D5: D_TVS, Diode_SMD:D_SOD-523, F.Cu at (126.1, 95.1)
- added RGB1: IN-P32TATRGB, pcb-Inolux:4-PLCC_3P2X2P8_INL, F.Cu at (165.7, 89.7)
- U5: renamed from U6; value AT93C46DN-SH-B -> 8S1_ATM
- moved R22 5.57 mm to (150.7, 94.3), turned to 0 degrees
- moved R23 5.44 mm to (148.8, 94.3), turned to 180 degrees
- moved C40 4.47 mm to (151.8, 88.2), turned to 180 degrees
- moved U6 3.63 mm to (147.3, 89.3), turned to 0 degrees
- moved R21 3.29 mm to (149.0, 88.2), turned to 180 degrees
- moved R7 2.38 mm to (149.8, 98.0), turned to 180 degrees
- moved J3 2.00 mm to (176.2, 90.9)
- moved J2 2.00 mm to (171.4, 90.9)
- moved R25 1.93 mm to (181.4, 88.8)
- moved R26 1.93 mm to (182.4, 88.8)
- moved C41 1.65 mm to (154.4, 96.0)
- moved X2 1.65 mm to (155.6, 97.6)
- moved C22 1.35 mm to (157.4, 99.1)
- moved C37 1.35 mm to (159.4, 99.9)
- moved C23 1.35 mm to (158.0, 98.5)
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- renumbered C25 to C17, C26 to C18, C27 to C19, C17 to C20, C18 to C21, C19 to C22, C20 to C23, C21 to C24, C22 to C25, C23 to C26, C24 to C27, C32 to C28, C28 to C29, C29 to C30, C30 to C31, C31 to C32, C40 to C39, C39 to C40, D7 to D10, D3 to D6, D4 to D7, D5 to D8, D6 to D9, J2 to J1, J1 to J2, J7 to J4, J9 to J7, J4 to J9, U7 to U6
Routing:
- net +1V8: track 109.7 -> 22.3 mm
- net /PGOOD1V2: track 1.46 -> 26.0 mm
- net /IOB_43a: track 0.00 -> 23.4 mm, vias 0 -> 2
- net /IOB_51a: track 0.00 -> 21.6 mm, vias 0 -> 2
- net /IOB_22a: track 0.00 -> 21.1 mm, vias 0 -> 2
- net /IOB_41a: track 0.00 -> 20.5 mm, vias 0 -> 2
- net /IOB_44b: track 0.00 -> 19.8 mm, vias 0 -> 2
- net /IOB_18a: track 0.00 -> 19.1 mm, vias 0 -> 2
- net /IOB_39a: track 0.00 -> 18.9 mm, vias 0 -> 2
- net /IOB_24a: track 0.00 -> 18.8 mm, vias 0 -> 2
- net /IOB_31b: track 0.00 -> 18.5 mm, vias 0 -> 2
- net /IOB_3b_G6: track 0.00 -> 18.2 mm, vias 0 -> 2
- net /IOB_37a: track 0.00 -> 17.5 mm, vias 0 -> 2
- net /IOB_13b: track 0.00 -> 17.5 mm, vias 0 -> 2
- net /IOB_29b: track 0.00 -> 17.4 mm, vias 0 -> 2
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- added copper zone on B.Cu, net GND
- added copper zone on In3.Cu, net GND
- added copper zone on In4.Cu, net GND
