File: designs/lattice-iCE40UP5K-SG48I/lattice-iCE40UP5K-SG48I.kicad_sch (KiCad schematic)
At the start: 89 parts, among them J1 USB_C_Receptacle_USB2.0_14P, J2 PRT-14417, J3 Conn_01x02, J4 Conn_01x07, J5 Conn_02x06_Top_Bottom, J6 Conn_02x06_Top_Bottom, J7 Conn_02x06_Top_Bottom, J8 Conn_02x06_Top_Bottom, SW1 SW_MEC_5G, U1 RTQ2520GQW, U2 RTQ2520GQW, U3 ICE40UP5K-SG48I, U4 FT2232HQ, U5 ESDR0502NMUTBG, U6 AT93C46DN-SH-B, U7 BY25Q40GWTIG, X1 DSC6003JI2B

Commit message: save
Parts:
- J5, J6, J7, J8: footprint Connector_PinHeader_2.54mm:PinHeader_2x06_P2.54mm_Vertical_SMD -> pcb-Samtec:SAMTEC-SMH-106-02-X-D
- renumbered R25 to R24
Changed lines of the file:
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@@
 		(in_pos_files yes)
 		(dnp no)
-		(property "Reference" "R25"
+		(property "Reference" "R24"
 			(at 536.956 194.31 0)
 			(show_name no)
@@
 			(project "lattice-iCE40UP5K-SG48I"
 				(path "/e0a68d80-6b92-4ac2-8789-569b9c117dc1"
-					(reference "R25")
+					(reference "R24")
 					(unit 1)
 				)
@@
 		(dnp no)
 		(fields_autoplaced yes)
-		(property "Reference" "#PWR072"
+		(property "Reference" "#PWR071"
 			(at 414.02 190.5 0)
 			(hide yes)
@@
 			(project "lattice-iCE40UP5K-SG48I"
 				(path "/e0a68d80-6b92-4ac2-8789-569b9c117dc1"
-					(reference "#PWR072")
+					(reference "#PWR071")
 					(unit 1)
 				)
@@
 		(dnp no)
 		(fields_autoplaced yes)
-		(property "Reference" "#PWR071"
+		(property "Reference" "#PWR070"
 			(at 129.54 190.5 0)
 			(hide yes)
@@
 			(project "lattice-iCE40UP5K-SG48I"
 				(path "/e0a68d80-6b92-4ac2-8789-569b9c117dc1"
-					(reference "#PWR071")
+					(reference "#PWR070")
 					(unit 1)
 				)
@@
 			)
 		)
-		(property "Footprint" "Connector_PinHeader_2.54mm:PinHeader_2x06_P2.54mm_Vertical_SMD"
+		(property "Footprint" "pcb-Samtec:SAMTEC-SMH-106-02-X-D"
 			(at 382.27 246.38 0)
 			(hide yes)
@@
 			)
 		)
-		(property "Footprint" "Connector_PinHeader_2.54mm:PinHeader_2x06_P2.54mm_Vertical_SMD"
+		(property "Footprint" "pcb-Samtec:SAMTEC-SMH-106-02-X-D"
 			(at 438.15 246.38 0)
 			(hide yes)
@@
 			)
 		)
-		(property "Footprint" "Connector_PinHeader_2.54mm:PinHeader_2x06_P2.54mm_Vertical_SMD"
+		(property "Footprint" "pcb-Samtec:SAMTEC-SMH-106-02-X-D"
 			(at 466.09 246.38 0)
 			(hide yes)
@@
 			)
 		)
-		(property "Footprint" "Connector_PinHeader_2.54mm:PinHeader_2x06_P2.54mm_Vertical_SMD"
+		(property "Footprint" "pcb-Samtec:SAMTEC-SMH-106-02-X-D"
 			(at 410.21 246.38 0)
 			(hide yes)
@@
 		(in_pos_files yes)
 		(dnp no)
-		(property "Reference" "#PWR070"
+		(property "Reference" "#PWR072"
 			(at 261.62 194.31 0)
 			(hide yes)
@@
 			(project "lattice-iCE40UP5K-SG48I"
 				(path "/e0a68d80-6b92-4ac2-8789-569b9c117dc1"
-					(reference "#PWR070")
+					(reference "#PWR072")
 					(unit 1)
 				)
