File: designs/lattice-iCE40UP5K-SG48I/lattice-iCE40UP5K-SG48I.kicad_sch (KiCad schematic)
At the start: 102 parts, among them J1 Conn_Coaxial_Small, J2 USB_C_Receptacle_USB2.0_14P, J4 PRT-14417, J5 Conn_02x06_Top_Bottom, J6 Conn_02x06_Top_Bottom, J7 Conn_01x02, J8 Conn_01x07, J9 Conn_02x06_Top_Bottom, SW1 SW_MEC_5G, U1 RTQ2520GQW, U2 RTQ2520GQW, U3 ICE40UP5K-SG48I, U4 FT2232HQ, U5 ESDR0502NMUTBG, U6 AT93C46DN-SH-B, U7 BY25Q40GWTIG, X1 DSC6003JI2B, X2 DSC6003JI2B

Commit message: ??
Parts:
- removed SW1: SW_MEC_5G, symbol Switch:SW_MEC_5G
- removed U5: ESDR0502NMUTBG, pcb-onsemi:ESDR0502NMUTBG, symbol pcb-onsemi:ESDR0502NMUTBG
- added D3, D4, D5: D_TVS, Diode_SMD:D_SOD-523, symbol Device:D_TVS
- added RGB1: IN-P32TATRGB, pcb-Inolux:4-PLCC_3P2X2P8_INL, symbol pcb-Inolux:IN-P32TATRGB
- renumbered C25 to C17, C26 to C18, C27 to C19, C17 to C20, C18 to C21, C19 to C22, C20 to C23, C21 to C24, C22 to C25, C23 to C26, C24 to C27, C32 to C28, C28 to C29, C29 to C30, C30 to C31, C31 to C32, C40 to C39, C39 to C40, D7 to D10, D3 to D6, D4 to D7, D5 to D8, D6 to D9, J2 to J1, J1 to J2, J7 to J4, J9 to J7, J4 to J9, U6 to U5, U7 to U6
Connections:
- net +3V3: now also RGB1.2 (VCC)
- net GND: now also D3.2 (A2), D4.2 (A2), D5.2 (A2)
- net RGB0: now also RGB1.1 (R)
- net RGB1: now also RGB1.3 (G)
- net RGB2: now also RGB1.4 (B)
- net USB_+: now also D5.1 (A1)
- net USB_-: now also D4.1 (A1)
- net VBUS: now also D3.1 (A1)
Other:
- note removed: "ADD A HEADER FOR FTDI PINS"
- note removed: "ADD ANOTHER PUSH BUTTON"
- moved on the sheet: C20, C21, C22, C23, C24, C25, C26, C27, C29, C30, C31, C32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
